File: Projet Banc Essai LCD/Projet Banc Essai LCD.kicad_pcb (KiCad board)
At the start: 2 copper layers, 14 parts

Commit message: mise à jour des fichiers
Other:
- board text added: "Projet Banc Essai LCD Lequette Kelan Conçu en France"
Changed lines of the file:
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@@
 		(embedded_fonts no)
+	)
+	(gr_text "Projet Banc Essai LCD\nLequette Kelan\nConçu en France"
+		(at 147.574 78.486 0)
+		(layer "F.SilkS")
+		(effects
+			(font
+				(size 1 1)
+				(thickness 0.1)
+			)
+			(justify bottom)
+		)
 	)
 	(segment

Commit message: mise à jour finale Kicad
Other:
- board outline added: 122.9 x 56.1 mm
Changed lines of the file:
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@@
 		(embedded_fonts no)
+	)
+	(gr_rect
+		(start 80.264 67.056)
+		(end 203.2 123.19)
+		(stroke
+			(width 0.05)
+			(type default)
+		)
+		(fill no)
+		(layer "Edge.Cuts")
 	)
 	(gr_text "Projet Banc Essai LCD\nLequette Kelan\nConçu en France"
